Commit message: adding odom_motion_model

File: src/servebot_description/urdf/servebot_urdf.xacro (robot description, xacro)
@@ -105,5 +105,5 @@
     <parent link="base_link"/>
     <child  link="caster_front_right"/>
-    <origin xyz="0.1975 -0.1625 0.04" rpy="0 0 0"/>
+    <origin xyz="0.1975 -0.1625 -0.015" rpy="0 0 0"/>
   </joint>
   <link name="caster_front_right">
@@ -116,5 +116,5 @@
     </inertial>
     <visual>
-      <origin xyz="0 0 0" rpy="-1.57 0 0"/>
+      <origin xyz="0 0 0.055" rpy="-1.57 0 0"/>
       <geometry>
         <mesh filename="package://servebot_description/meshes/caster_front_right.stl" scale="0.001 0.001 0.001"/>
@@ -135,5 +135,5 @@
     <parent link="base_link"/>
     <child  link="caster_front_left"/>
-    <origin xyz="0.1975 0.1625 0.04" rpy="0 0 0"/>
+    <origin xyz="0.1975 0.1625 -0.015" rpy="0 0 0"/>
   </joint>
   <link name="caster_front_left">
@@ -146,5 +146,5 @@
     </inertial>
     <visual>
-      <origin xyz="0 0 0" rpy="-1.57 0 0"/>
+      <origin xyz="0 0 0.055" rpy="-1.57 0 0"/>
       <geometry>
         <mesh filename="package://servebot_description/meshes/caster_front_left.stl" scale="0.001 0.001 0.001"/>
@@ -165,5 +165,5 @@
     <parent link="base_link"/>
     <child  link="caster_rear_right"/>
-    <origin xyz="-0.1975 -0.1625 0.04" rpy="0 0 0"/>
+    <origin xyz="-0.1975 -0.1625 -0.015" rpy="0 0 0"/>
   </joint>
   <link name="caster_rear_right">
@@ -176,5 +176,5 @@
     </inertial>
     <visual>
-      <origin xyz="0 0 0" rpy="-1.57 0 0"/>
+      <origin xyz="0 0 0.055" rpy="-1.57 0 0"/>
       <geometry>
         <mesh filename="package://servebot_description/meshes/caster_rear_right.stl" scale="0.001 0.001 0.001"/>
@@ -195,5 +195,5 @@
     <parent link="base_link"/>
     <child  link="caster_rear_left"/>
-    <origin xyz="-0.1975 0.1625 0.04" rpy="0 0 0"/>
+    <origin xyz="-0.1975 0.1625 -0.015" rpy="0 0 0"/>
   </joint>
   <link name="caster_rear_left">
@@ -206,5 +206,5 @@
     </inertial>
     <visual>
-      <origin xyz="0 0 0" rpy="-1.57 0 0"/>
+      <origin xyz="0 0 0.055" rpy="-1.57 0 0"/>
       <geometry>
         <mesh filename="package://servebot_description/meshes/caster_rear_left.stl" scale="0.001 0.001 0.001"/>

Commit message: new base link and other sensor links

File: src/servebot_description/urdf/servebot_urdf.xacro (robot description, xacro)
@@ -33,7 +33,7 @@
     </visual>
     <collision>
-      <origin xyz="0.0 0.0 0.096" rpy="0 0 0"/>
-      <geometry>
-        <box size="0.45 0.35 0.20"/>
+      <origin xyz="0.0 0.0 0.037" rpy="0 0 0"/>
+      <geometry>
+        <box size="0.45 0.445 0.020"/>
       </geometry>
     </collision>
@@ -246,8 +246,38 @@
   </link>
   <joint name="imu_joint" type="fixed">
-    <origin xyz="0 0 0.119" rpy="0 0 0" />
+    <origin xyz="0 0 0.10" rpy="0 0 0" />
     <parent link="base_link" />
     <child link="imu_link" />
     <axis xyz="0 0 0" />
   </joint>
+  <link name="laser_link">
+    <inertial>
+      <origin xyz="-0.011945780406062 -0.000381929217680526 -0.0170649378129477" rpy="0 0 0" />
+      <mass value="0.073084435549317" />
+      <inertia ixx="1.96074931730795E-05" ixy="-3.62091076640009E-07" ixz="4.28230084046735E-07"
+               iyy="2.40983835136327E-05" iyz="1.50180909250652E-08"
+               izz="4.14184164228595E-05" />
+    </inertial>
+    <visual>
+      <origin xyz="0 0 0" rpy="0 0 0" />
+      <geometry>
+        <mesh filename="package://servebot_description/meshes/laser_link.STL" />
+      </geometry>
+      <material name="dark_grey">
+        <color rgba="0.2 0.2 0.2 1.0"/>
+      </material>
+    </visual>
+    <collision>
+      <origin xyz="0 0 0" rpy="0 0 0" />
+      <geometry>
+        <cylinder radius="0.040" length="0.040"/>
+      </geometry>
+    </collision>
+  </link>
+  <joint name="laser_joint" type="fixed">
+    <origin xyz="-0.0050526 -0.0023221 0.1208" rpy="0 0 3.14" />
+    <parent link="base_link" />
+    <child link="laser_link" />
+    <axis xyz="0 0 0" />
+  </joint>
 </robot>
