Commit message: Migrate from Ignition to Gazebo Harmonic - update plugins, collision shapes, bridge topics

File: src/servebot_description/urdf/servebot_gazebo.xacro (robot description, xacro)
@@ -54,5 +54,5 @@
   </gazebo>
   <gazebo>
-      <plugin filename="ign_ros2_control-system" name="ign_ros2_control::IgnitionROS2ControlPlugin">
+      <plugin filename="gz_ros2_control-system" name="gz_ros2_control::GazeboSimROS2ControlPlugin">
         <parameters>$(find servebot_controller)/config/servebot_controllers.yaml</parameters>
       </plugin>

File: src/servebot_description/urdf/servebot_ros2_control.xacro (robot description, xacro)
@@ -1,5 +1,5 @@
 <?xml version="1.0"?>
 <robot xmlns:xacro="http://www.ros.org/wiki/xacro" name="servebot">
-    <!-- sim_mode=true  → ign_ros2_control (Gazebo)              -->
+    <!-- sim_mode=true  → gz_ros2_control (Gazebo Harmonic)      -->
     <!-- sim_mode=false → servebot_firmware/ServebotInterface (ESP32) -->
     <xacro:arg name="sim_mode" default="true"/>
@@ -7,5 +7,5 @@
         <hardware>
             <xacro:if value="$(arg sim_mode)">
-                <plugin>ign_ros2_control/IgnitionSystem</plugin>
+                <plugin>gz_ros2_control/GazeboSimSystem</plugin>
             </xacro:if>
             <xacro:unless value="$(arg sim_mode)">

File: src/servebot_description/urdf/servebot_urdf.xacro (robot description, xacro)
@@ -33,7 +33,7 @@
     </visual>
     <collision>
-      <origin xyz="0.0 0.0 0.0" rpy="0 0 0"/>
-      <geometry>
-        <mesh filename="package://servebot_description/meshes/base_link.stl" scale="0.001 0.001 0.001"/>
+      <origin xyz="0.0 0.0 0.096" rpy="0 0 0"/>
+      <geometry>
+        <box size="0.45 0.35 0.20"/>
       </geometry>
     </collision>
@@ -64,7 +64,7 @@
     </visual>
     <collision>
-      <origin xyz="0.0 0.0 0.0" rpy="3.14 0 0"/>
-      <geometry>
-        <mesh filename="package://servebot_description/meshes/wheel_right.stl" scale="0.001 0.001 0.001"/>
+      <origin xyz="0.0 0.0 0.0" rpy="1.5707 0 0"/>
+      <geometry>
+        <cylinder radius="0.060" length="0.040"/>
       </geometry>
     </collision>
@@ -95,7 +95,7 @@
     </visual>
     <collision>
-       <origin xyz="0.0 0.0 0.0" rpy="0 0 0"/>
-      <geometry>
-        <mesh filename="package://servebot_description/meshes/wheel_left.stl" scale="0.001 0.001 0.001"/>
+      <origin xyz="0.0 0.0 0.0" rpy="1.5707 0 0"/>
+      <geometry>
+        <cylinder radius="0.060" length="0.040"/>
       </geometry>
     </collision>
@@ -125,7 +125,7 @@
     </visual>
     <collision>
-      <origin xyz="0 0 0" rpy="-1.57 0 0"/>
-      <geometry>
-        <mesh filename="package://servebot_description/meshes/caster_front_right.stl" scale="0.001 0.001 0.001"/>
+      <origin xyz="0 0 0" rpy="0 0 0"/>
+      <geometry>
+        <sphere radius="0.022"/>
       </geometry>
     </collision>
@@ -155,7 +155,7 @@
     </visual>
     <collision>
-      <origin xyz="0 0 0" rpy="-1.57 0 0"/>
-      <geometry>
-        <mesh filename="package://servebot_description/meshes/caster_front_left.stl" scale="0.001 0.001 0.001"/>
+      <origin xyz="0 0 0" rpy="0 0 0"/>
+      <geometry>
+        <sphere radius="0.022"/>
       </geometry>
     </collision>
@@ -185,7 +185,7 @@
     </visual>
     <collision>
-      <origin xyz="0 0 0" rpy="-1.57 0 0"/>
-      <geometry>
-        <mesh filename="package://servebot_description/meshes/caster_rear_right.stl" scale="0.001 0.001 0.001"/>
+      <origin xyz="0 0 0" rpy="0 0 0"/>
+      <geometry>
+        <sphere radius="0.022"/>
       </geometry>
     </collision>
@@ -215,7 +215,7 @@
     </visual>
     <collision>
-      <origin xyz="0 0 0" rpy="-1.57 0 0"/>
-      <geometry>
-        <mesh filename="package://servebot_description/meshes/caster_rear_left.stl" scale="0.001 0.001 0.001"/>
+      <origin xyz="0 0 0" rpy="0 0 0"/>
+      <geometry>
+        <sphere radius="0.022"/>
       </geometry>
     </collision>
@@ -241,5 +241,5 @@
       <origin xyz="0 0 0" rpy="0 0 0" />
       <geometry>
-        <mesh filename="package://servebot_description/meshes/imu_link.STL" />
+        <box size="0.02 0.02 0.01"/>
       </geometry>
     </collision>

Commit message: Add laser lidar, twist_mux teleop, and twist_relay nodes
- servebot_urdf.xacro: fix laser_link mesh ref (bumperbot→servebot),
  replace mesh collision with cylinder, fix visual origin offset
- servebot_gazebo.xacro: add gpu_lidar sensor with Sensors system plugin,
  set visualize=false for performance
- gazebo.launch.py: bridge /scan topic (LaserScan) to ROS2
- twist_relay.py / twist_relay.cpp: Twist↔TwistStamped relay for
  servebot_controller, fix bumperbot topic refs, add frame_id
- joystick_teleop.launch.py: fix missing imports, add twist_mux and
  twist_relay to launch, fix cmd_vel_out to /cmd_vel
- joy_teleop.yaml: publish plain Twist to joy_vel via twist_mux
- twist_mux_topics/locks/joy.yaml: add twist_mux config files
- CMakeLists.txt: register twist_relay executable

File: src/servebot_description/urdf/servebot_gazebo.xacro (robot description, xacro)
@@ -57,4 +57,7 @@
         <parameters>$(find servebot_controller)/config/servebot_controllers.yaml</parameters>
       </plugin>
+      <plugin filename="gz-sim-sensors-system" name="gz::sim::systems::Sensors">
+        <render_engine>ogre2</render_engine>
+      </plugin>
   </gazebo>
   <gazebo reference="imu_link">
@@ -108,3 +111,33 @@
     </sensor>
   </gazebo>
+  <!-- 2D Laser Sensor -->
+  <gazebo reference="laser_link">
+    <sensor name="lidar" type="gpu_lidar">
+      <always_on>true</always_on>
+      <visualize>false</visualize>
+      <topic>scan</topic>
+      <update_rate>5</update_rate>
+      <gz_frame_id>laser_link</gz_frame_id>
+      <lidar>
+        <scan>
+          <horizontal>
+            <samples>360</samples>
+            <resolution>1.00000</resolution>
+            <min_angle>0.000000</min_angle>
+            <max_angle>6.280000</max_angle>
+          </horizontal>
+        </scan>
+        <range>
+          <min>0.120000</min>
+          <max>12.0</max>
+          <resolution>0.02</resolution>
+        </range>
+        <noise>
+          <type>gaussian</type>
+          <mean>0.0</mean>
+          <stddev>0.01</stddev>
+        </noise>
+      </lidar>
+    </sensor>
+  </gazebo>
 </robot>

File: src/servebot_description/urdf/servebot_urdf.xacro (robot description, xacro)
@@ -35,5 +35,5 @@
       <origin xyz="0.0 0.0 0.037" rpy="0 0 0"/>
       <geometry>
-        <box size="0.45 0.445 0.020"/>
+        <box size="0.445 0.445 0.020"/>
       </geometry>
     </collision>
